File: digout.kicad_sch (KiCad schematic)
At the start: 16 parts, among them U22 TXUN0104RUTR, U23 ADUM5240ARZ, U24 ADUM5240ARZ

Commit message: Add DCCT ADCs
Parts:
- removed C100, C102, C103, C104, C99: 0.1uF, Capacitor_SMD:C_0402_1005Metric, symbol Device:C_Small
- removed C101, C98: 10uF, Capacitor_SMD:C_0603_1608Metric, symbol Device:C_Small
- removed CR1, CR2: SP3006-02XTG, myparts:SOT563_LTF, symbol PSC:SP3006-02XTG
- removed R34, R35, R36, R37: 2.49K, Resistor_SMD:R_0402_1005Metric, symbol Device:R_US
- added C182, C183, C184, C185, C186: 0.1uF, Capacitor_SMD:C_0402_1005Metric, symbol Device:C_Small
- added C187, C188: 10uF, Capacitor_SMD:C_0603_1608Metric, symbol Device:C_Small
- added CR5, CR6: SP3006-02XTG, myparts:SOT563_LTF, symbol PSC:SP3006-02XTG
- added R66, R67, R68, R69: 2.49K, Resistor_SMD:R_0402_1005Metric, symbol Device:R_US
- U39: renamed from U23; footprint myparts:R_8_ADI-M -> myparts:R_8_ADI
- U40: renamed from U24; footprint myparts:R_8_ADI-M -> myparts:R_8_ADI
- renumbered U22 to U38
Connections:
- net +1V8: now also C182.1
- net +5V: now also C183.1, C184.1
- net GND: now also C182.2, C183.2, C184.2, C185.2, C186.2, C187.2, C188.2
- net dout0_iso: now also CR5.1, R66.1
- net dout1_iso: now also CR5.5, R68.1
- net dout2_iso: now also CR6.1, R67.1
- net dout3_iso: now also CR6.5, R69.1
- net dout_iso_gnd: now also CR5.2, CR5.4, CR6.2, CR6.4
- net at U39.8 (VISO): now also C185.1, C187.1, R66.2, R68.2
- net at U40.8 (VISO): now also C186.1, C188.1, R67.2, R69.2

Commit message: DAC and DCCT placement
Connections:
- net +1V8 renamed +1.8V
Changed lines of the file:
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@@
-	)
-	(symbol
-		(lib_id "power:+1V8")
-		(at 36.83 74.93 0)
-		(unit 1)
-		(exclude_from_sim no)
-		(in_bom yes)
-		(on_board yes)
-		(dnp no)
-		(fields_autoplaced yes)
-		(property "Reference" "#PWR0264"
-			(at 36.83 78.74 0)
-			(effects
-				(font
-					(size 1.27 1.27)
-				)
-				(hide yes)
-			)
-		)
-		(property "Value" "+1V8"
-			(at 36.83 69.85 0)
-			(effects
-				(font
-					(size 1.27 1.27)
-				)
-			)
-		)
-		(property "Footprint" ""
-			(at 36.83 74.93 0)
-			(effects
-				(font
-					(size 1.27 1.27)
-				)
-				(hide yes)
-			)
-		)
-		(property "Datasheet" ""
-			(at 36.83 74.93 0)
-			(effects
-				(font
-					(size 1.27 1.27)
-				)
-				(hide yes)
-			)
-		)
-		(property "Description" "Power symbol creates a global label with name \"+1V8\""
-			(at 36.83 74.93 0)
-			(effects
-				(font
-					(size 1.27 1.27)
-				)
-				(hide yes)
-			)
-		)
-		(pin "1"
-		)
-		(instances
-			(project "psc_daughter_brd"
-				(path "/40891cc8-bf64-41f4-8f69-a607d7b280eb/979dab62-5512-4152-97ee-117138a961d3/84c3e299-56b9-4043-9091-ed3bb176fd4f"
-					(reference "#PWR0264")
-					(unit 1)
-				)
-			)
-		)
 	)
 	(symbol
@@
 					(unit 1)
 				)
+			)
+		)
+	)
+	(symbol
+		(lib_id "PSC:+1.8V")
+		(at 36.83 74.93 0)
+		(unit 1)
+		(exclude_from_sim no)
+		(in_bom yes)
+		(on_board yes)
+		(dnp no)
+		(fields_autoplaced yes)
+		(property "Reference" "#PWR0161"
+			(at 36.83 78.74 0)
+			(effects
+				(font
+					(size 1.27 1.27)
+				)
+				(hide yes)
+			)
+		)
+		(property "Value" "+1.8V"
+			(at 36.83 69.85 0)
+			(effects
+				(font
+					(size 1.27 1.27)
+				)
+			)
+		)
+		(property "Footprint" ""
+			(at 36.83 74.93 0)
+			(effects
+				(font
+					(size 1.27 1.27)
+				)
+				(hide yes)
+			)
+		)
+		(property "Datasheet" ""
+			(at 36.83 74.93 0)
+			(effects
+				(font
+					(size 1.27 1.27)
+				)
+				(hide yes)
+			)
+		)
+		(property "Description" ""
+			(at 36.83 74.93 0)
+			(effects
+				(font
+					(size 1.27 1.27)
+				)
+				(hide yes)
+			)
+		)
+		(pin "1"
+		)
+		(instances
+			(project "psc_daughter_brd"
+				(path "/40891cc8-bf64-41f4-8f69-a607d7b280eb/979dab62-5512-4152-97ee-117138a961d3/84c3e299-56b9-4043-9091-ed3bb176fd4f"
+					(reference "#PWR0161")
+					(unit 1)
+				)

Commit message: Finish layout
Parts:
- added C104: 0.1uF, Capacitor_SMD:C_0402_1005Metric, symbol Device:C_Small
- C182, C183, C184, C185, C186: MFG (none) -> Taiyo Yuden; MFG_PN (none) -> TMK105BJ104KV-F
- C187, C188: MFG (none) -> Samsung; MFG_PN (none) -> CL10A106MA8NRNC
- CR5, CR6: Cost (none) -> 0.65; MFG (none) -> Littlefuse; MFG_PN (none) -> SP3006-02XTG
- R66, R67, R68, R69: Cost (none) -> .01; MFG (none) -> Panasonic; MFG_PN (none) -> ERJ-2RKF2491X
- U38: Cost (none) -> .77; MFG (none) -> TI; MFG_PN (none) -> TXUN0104RUTR
- U39, U40: footprint myparts:R_8_ADI -> myparts:R_8_ADI-M; Cost (none) -> 6.81; MFG (none) -> Analog Devices; MFG_PN (none) -> ADUM5240ARZ
Connections:
- net GND: now also C104.2
- net +5V renamed +5.0V
- net +5.0V: now also C104.1
Other:
- moved on the sheet: C183
