File: monitor_fe.kicad_sch (KiCad schematic)
At the start: 18 parts, among them U12 AD8221, U13 OPA277

Commit message: Add DCCT ADCs
Parts:
- renumbered C43 to C1, C52 to C10, C44 to C2, C45 to C3, C46 to C4, C47 to C5, C48 to C6, C49 to C7, C50 to C8, C51 to C9, R10 to R1, R11 to R2, R12 to R3, R13 to R4, R14 to R5, R15 to R6, U12 to U1, U13 to U2

Commit message: Finish layout
Parts:
- added C101: 2200pF, myparts:EMCT101W222M1GV001E, symbol PSC:EMCT101W222M1GV001E
- added D2: SP3118-01ETG, myparts:sp3118-01etg, symbol PSC:SP3118-01ETG
- C1: Cost (none) -> .01; MFG (none) -> Kemet; MFG_PN (none) -> C0402C221K5RACTU
- C10, C4, C5, C9: MFG (none) -> Taiyo Yuden; MFG_PN (none) -> TMK105BJ104KV-F
- C2, C3, C6, C7: MFG (none) -> Samsung; MFG_PN (none) -> CL10A106MA8NRNC
- C8: MFG (none) -> Samsung; MFG_PN (none) -> CL05B472KB5NNNC
- R1, R2: value 1K -> 1.0K; Cost (none) -> .01; MFG (none) -> Panasonic; MFG_PN (none) -> ERJ-2RKF1001X
- R3: MFG (none) -> Panasonic; MFG_PN (none) -> ERJ-2RKF10R0X; now not fitted
- R4, R5: Cost (none) -> .01; MFG (none) -> Panasonic; MFG_PN (none) -> ERJ-2RKF1002X
- R6: Cost (none) -> .01; MFG (none) -> Panasonic; MFG_PN (none) -> ERJ-2RKF10R0X
- U1: Cost (none) -> 10.23; MFG (none) -> Analog Devices; MFG_PN (none) -> AD8221BRZ
- U2: Cost (none) -> 2.66; MFG (none) -> Analog Devices; MFG_PN (none) -> OPA277UA/2K5
Connections:
- net GND: now also C101.3, C101.4
- net at C1.1, R1.1, U1.4 (+): now also C101.1, D2.2 (A2)
- net at C1.2, R2.1, U1.1 (-): now also C101.2, D2.1 (A1)
Other:
- moved on the sheet: C1, R1, R2
