File: psc_daughter_brd.kicad_sch (KiCad schematic)
At the start: 4 parts

Commit message: Change DAC outputs to 1.8v
Other:
- title: Power Supply Controller -> Power Supply Controller Daughterboard
Changed lines of the file:
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@@
 	(paper "B")
 	(title_block
-		(title "Power Supply Controller")
+		(title "Power Supply Controller Daughterboard")
 		(date "2025-11-21")
 		(company "BNL")

Commit message: Finish layout
Parts:
- added TP2, TP3, TP4, TP5: ${SHORT_NET_NAME(1)}, myparts:TestPoint_RCS-0C, symbol Connector:TestPoint
Connections:
- net GND: now also TP2.1, TP3.1, TP4.1, TP5.1
